File: hardware/pcbs/tile_light_pcb/tile_light_pcb.kicad_pcb (KiCad board)
At the start: 2 copper layers, 47 x 27 mm, 33 parts, among them CN1 ZX-ZH1.5-5PLT, CN2 ZX-ZH1.5-5PLT, CN3 ZX-ZH1.5-2PLT

Commit message: hardware: tile light pcb: Added buttons and did routing
Parts:
- removed C10, C6: 100nF, Capacitor_SMD:C_0402_1005Metric
- removed LED10, LED6: SK6812MINIRGBW-WS-P6-A, openstw:LED-SMD_6P-L3.5-W3.5_SK6812MINIRGBW-WS-P6-A
- added CN4: ZX-ZH1.5-2PLT, openstw:CONN-SMD_2P-P1.50_ZX-ZH1.5-2PLT, B.Cu at (132.8, 91.1)
- added CN5: ZX-ZH1.5-2PLT, openstw:CONN-SMD_2P-P1.50_ZX-ZH1.5-2PLT, B.Cu at (147.5, 91.1)
- added SW1: HX-6X6X7.3-TP FT SQUARE BUTTON, openstw:SW-SMD_4P-L6.0-W6.0-P4.50-LS9.0-H7.3, F.Cu at (122.2, 99.2)
- added SW2: HX-6X6X7.3-TP FT SQUARE BUTTON, openstw:SW-SMD_4P-L6.0-W6.0-P4.50-LS9.0-H7.3, F.Cu at (158.2, 99.2)
- moved C8 3.79 mm to (142.8, 99.0), turned to 90 degrees
- moved C7 3.67 mm to (133.9, 99.2), turned to 90 degrees
- moved C9 3.61 mm to (146.6, 99.2), turned to -90 degrees
- turned LED7 to 90 degrees
- turned LED8 to 90 degrees
- turned LED9 to -90 degrees
Connections:
- LED11 pad 3: Net-(LED10-DOUT) -> Net-(LED11-DIN)
- LED7 pad 3: Net-(LED6-DOUT) -> Net-(LED5-DOUT)
- LED9 pad 5: Net-(LED10-DIN) -> Net-(LED11-DIN)
Routing:
- net +5V: track 0.00 -> 220.1 mm, vias 0 -> 5
- net GND: track 0.00 -> 62.2 mm, vias 0 -> 35
- net LED_DIN: track 0.00 -> 46.3 mm, vias 0 -> 1
- net LED_DOUT: track 0.00 -> 43.5 mm, vias 0 -> 7
- net Net-(LED5-DOUT): track 0.00 -> 43.1 mm, vias 0 -> 4
- net Net-(LED11-DIN): track 0.00 -> 38.4 mm, vias 0 -> 8
- net BTN2: track 0.00 -> 17.0 mm, vias 0 -> 1
- net BTN1: track 0.00 -> 14.4 mm, vias 0 -> 1
- net Net-(LED7-DOUT): track 0.00 -> 12.9 mm
- net Net-(LED8-DOUT): track 0.00 -> 9.09 mm
- net Net-(LED13-DOUT): track 0.00 -> 6.20 mm
- net Net-(LED3-DOUT): track 0.00 -> 6.08 mm
- net Net-(LED4-DOUT): track 0.00 -> 6.06 mm
- net Net-(LED2-DOUT): track 0.00 -> 6.06 mm
- net Net-(LED14-DOUT): track 0.00 -> 6.06 mm
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- added copper zone on B.Cu, net GND
- added copper zone on F.Cu, net GND
Other:
- board text added: "+5V GND"
- board text added: "- + D + -"
- board text added: "BTN1"
- board text added: "BTN2"
- board text added: "GND SIG"
- board text added: "POWER"
